File: hardware/heatvalve-6-rev2.1/heatvalve-6-rev2.1.kicad_sch (KiCad schematic)
At the start: 103 parts, among them J1 USB4105-GF-A, J10 ONEWIRE 3, J11 I2C EXPANSION DNP, J2 MOTOR 1 4P4C, J3 MOTOR 2 4P4C, J4 MOTOR 3 4P4C, J5 MOTOR 4 4P4C, J6 MOTOR 5 4P4C, J7 MOTOR 6 4P4C, J8 ONEWIRE 1, J9 ONEWIRE 2, SW1 RESET, SW2 BOOT, U1 ESP32-S3-WROOM-1-N16R8, U10 MCP6004, U11 LM339B, U12 74HC74, U2 USBLC6-2SC6, U21 DRV8837DSGR, U22 DRV8837DSGR, U23 DRV8837DSGR, U24 DRV8837DSGR, U25 DRV8837DSGR, U26 DRV8837DSGR, U3 MT2492, U9 INA180A1 (x20)

Commit message: Add measurement and position model documentation for Rev 2.1
This commit introduces a new markdown file detailing the current, BEMF, engagement, and position model for the Rev 2.1 hardware. The document outlines the purpose of separating force measurement from motion measurement, describes mechanical landmarks, pin-engagement recognition, candidate tacho qualification, endstop and fault classification, flow mapping, and prototype gate considerations. It also includes references for further reading on sensorless position control and related topics.
Parts:
- removed C15: 100n, Capacitor_SMD:C_0603_1608Metric, symbol Device:C
- removed C16: 100n DNP, Capacitor_SMD:C_0603_1608Metric, symbol Device:C
- removed R17, R18: 100k, Resistor_SMD:R_0603_1608Metric, symbol Device:R
- removed R19: 2.2k, Resistor_SMD:R_0603_1608Metric, symbol Device:R
- removed R20, R22: 10k, Resistor_SMD:R_0603_1608Metric, symbol Device:R
- removed R21: 1M, Resistor_SMD:R_0603_1608Metric, symbol Device:R
- added C50, C51, C53: 100n, Capacitor_SMD:C_0603_1608Metric, symbol Device:C
- added C52: 4.7n, Capacitor_SMD:C_0603_1608Metric, symbol Device:C
- added C54: 100n DNP, Capacitor_SMD:C_0603_1608Metric, symbol Device:C
- added D7: BAT54S BEMF ADC clamp, Package_TO_SOT_SMD:SOT-23, symbol Diode:BAT54S
- added R50, R52: 90.9k 1%, Resistor_SMD:R_0603_1608Metric, symbol Device:R
- added R51, R53: 47k 1%, Resistor_SMD:R_0603_1608Metric, symbol Device:R
- added R54: 1k, Resistor_SMD:R_0603_1608Metric, symbol Device:R
- added R55, R57, R60, R61, R62: 100k, Resistor_SMD:R_0603_1608Metric, symbol Device:R
- added R56, R59, R70, R71, R72, R73, R74, R75, R76, R77, R78, R79, R80, R81: 10k, Resistor_SMD:R_0603_1608Metric, symbol Device:R
- added R58: 1M, Resistor_SMD:R_0603_1608Metric, symbol Device:R
- added U13, U14: 74HC4051, Package_SO:TSSOP-16_4.4x5mm_P0.65mm, symbol 74xx:74HC4051
- R24: value 9.1k -> 18k
- RSH1: value 2.2R 1% -> 1.0R 1%; MPN 2.2R 1206 1% -> 1.0R 1206 1%
Connections:
- net +3V3_A: now also C50.1, C51.1, D7.2 (K), U13.16 (VCC), U14.16 (VCC)
- net +3V3_SYS: now also R59.1
- net GND: now also C50.2, C51.2, C52.2, D7.1 (A), R60.2, R61.2, R62.2, U13.2 (A6), U13.4 (A7), U13.6 (~{E}), U13.7 (VEE), U13.8 (GND), U14.2 (A6), U14.4 (A7), U14.6 (~{E}), U14.7 (VEE), U14.8 (GND)
- net MOT1_A: now also R70.1
- net MOT1_B: now also R71.1
- net MOT2_A: now also R72.1
- net MOT2_B: now also R73.1
- net MOT3_A: now also R74.1
- net MOT3_B: now also R75.1
- net MOT4_A: now also R76.1
- net MOT4_B: now also R77.1
- net MOT5_A: now also R78.1
- net MOT5_B: now also R79.1
- net MOT6_A: now also R80.1
- net MOT6_B: now also R81.1
- net TACHO_EDGE: now also R58.1, R59.2
- net VBIAS: now also R53.2, R55.2, R56.2; no longer U10.12 (+)
- net BEMF_SEL2: now reaches U1.12 (IO8)
- net BEMF_SEL2: now also R62.1, U13.9 (S2), U14.9 (S2)
- net ADC_BEMF: now reaches U1.5 (IO5)
- net ADC_BEMF: now also C52.1, D7.3 (COM), R54.2
- net BEMF_SEL0: now reaches U1.6 (IO6)
- net BEMF_SEL0: now also R60.1, U13.11 (S0), U14.11 (S0)
- net BEMF_SEL1: now reaches U1.7 (IO7)
- net BEMF_SEL1: now also R61.1, U13.10 (S1), U14.10 (S1)
- net OP_SPARE renamed BEMF_GAIN_FB
- net BEMF_GAIN_FB: now also R56.1, R57.2; no longer U10.14
- net TACHO_AMP renamed BEMF_RAW
- net BEMF_RAW: now also C53.1, C54.1, R51.1, R54.1
- net TACHO_CMP renamed BEMF_TACH_AMP
- net BEMF_TACH_AMP: now also U10.14, R57.1, R58.2
- net TAC_FB renamed BEMF_DIFF_N
- net BEMF_DIFF_N: now also R50.2, R51.2
- net TAC_IN renamed BEMF_DIFF_P
- net BEMF_DIFF_P: now also R52.2, R53.1
- new net BEMF_A1: R70.2, U13.13 (A0)
- new net BEMF_A2: R72.2, U13.14 (A1)
- new net BEMF_A3: R74.2, U13.15 (A2)
- new net BEMF_A4: R76.2, U13.12 (A3)
- new net BEMF_A5: R78.2, U13.1 (A4)
- new net BEMF_A6: R80.2, U13.5 (A5)
- new net BEMF_AC: C53.2, C54.2, R55.1, U10.12 (+)
- new net BEMF_B1: R71.2, U14.13 (A0)
- new net BEMF_B2: R73.2, U14.14 (A1)
- new net BEMF_B3: R75.2, U14.15 (A2)
- new net BEMF_B4: R77.2, U14.12 (A3)
- new net BEMF_B5: R79.2, U14.1 (A4)
- new net BEMF_B6: R81.2, U14.5 (A5)
- new net BEMF_MUX_A: R50.1, U13.3 (A)
- new net BEMF_MUX_B: R52.1, U14.3 (A)
- no-connect marks 31 -> 27
Other:
- note added: "30mA=0.60V, 60mA=1.20V, 150mA=3.00V. Engagement current remains measurable."
- note added: "ADC_BEMF is differential motion evidence; TACHO_EDGE counts qualified commutation."
- note added: "SELECTED DIFFERENTIAL BEMF / TACHO"
- note added: "SHARED SHUNT / CURRENT"
- note removed: "30mA=1.32V, 60mA=2.64V. ADC saturation above ~70mA is intentional."
- note removed: "SHARED SHUNT / CURRENT / TACHO"
